File: board/left_board/mcu_powsup.kicad_sch (KiCad schematic)
At the start: 5 parts

Commit message: left board: fix cap: 4.7nF -> 4.7µF
Parts:
- C701: LCSC C1538 -> C23733
Changed lines of the file:
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@@
 			)
 		)
-		(property "LCSC" "C1538"
+		(property "LCSC" "C23733"
 			(at 76.2 49.53 0)
 			(effects
