File: board/left_board/mcu.kicad_sch (KiCad schematic)
At the start: 2 parts, among them J401 UART, U401 STM32G0B0CETx

Commit message: left: replace UART pin header
choose a 2.54mm variant that can be mounted easily
Parts:
- J401: footprint Connector_PinHeader_2.54mm:PinHeader_2x01_P2.54mm_Vertical_SMD -> Connector_PinHeader_2.54mm:PinHeader_1x02_P2.54mm_Vertical_SMD_Pin1Left; LCSC C2883176 -> C5160785
Changed lines of the file:
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@@
 			)
 		)
-		(property "Footprint" "Connector_PinHeader_2.54mm:PinHeader_2x01_P2.54mm_Vertical_SMD"
+		(property "Footprint" "Connector_PinHeader_2.54mm:PinHeader_1x02_P2.54mm_Vertical_SMD_Pin1Left"
 			(at 163.83 67.31 0)
 			(effects
@@
 			)
 		)
-		(property "LCSC" "C2883176"
+		(property "LCSC" "C5160785"
 			(at 163.83 67.31 0)
 			(effects
